File: timagotchi-pcb/timagotchi-pcb.kicad_sch (KiCad schematic)
At the start: 8 parts, among them SW1 SW_Push, SW2 SW_Push

Commit message: use pwr_flag correctly, start pcb
Connections:
- net +9V: now reaches U1.30 (VIN)
- net GND renamed -BATT
Changed lines of the file:
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@@
   (junction (at 165.735 82.55) (diameter 0) (color 0 0 0 0)
   )
+  (junction (at 163.195 80.01) (diameter 0) (color 0 0 0 0)
+  )
   (junction (at 106.045 81.28) (diameter 0) (color 0 0 0 0)
+  )
+  (junction (at 163.195 68.58) (diameter 0) (color 0 0 0 0)
+  )
+  (junction (at 165.735 68.58) (diameter 0) (color 0 0 0 0)
   )
   (junction (at 106.045 106.68) (diameter 0) (color 0 0 0 0)
@@
     (stroke (width 0) (type default) (color 0 0 0 0))
   )
+  (wire (pts (xy 163.195 80.01) (xy 169.545 80.01))
+    (stroke (width 0) (type default) (color 0 0 0 0))
+  )
   (wire (pts (xy 160.655 95.25) (xy 172.085 95.25))
     (stroke (width 0) (type default) (color 0 0 0 0))
   )
-  (wire (pts (xy 163.195 65.405) (xy 163.195 80.01))
-    (stroke (width 0) (type default) (color 0 0 0 0))
-  )
-  (wire (pts (xy 165.735 82.55) (xy 165.735 65.405))
+  (wire (pts (xy 163.195 65.405) (xy 163.195 68.58))
+    (stroke (width 0) (type default) (color 0 0 0 0))
+  )
+  (wire (pts (xy 165.735 82.55) (xy 165.735 68.58))
     (stroke (width 0) (type default) (color 0 0 0 0))
   )
@@
     (stroke (width 0) (type default) (color 0 0 0 0))
   )
+  (wire (pts (xy 165.735 68.58) (xy 165.735 65.405))
+    (stroke (width 0) (type default) (color 0 0 0 0))
+  )
   (wire (pts (xy 118.745 106.68) (xy 106.045 106.68))
     (stroke (width 0) (type default) (color 0 0 0 0))
@@
     (stroke (width 0) (type default) (color 0 0 0 0))
   )
+  (wire (pts (xy 163.195 68.58) (xy 163.195 80.01))
+    (stroke (width 0) (type default) (color 0 0 0 0))
+  )
   (wire (pts (xy 106.045 106.68) (xy 106.045 112.395))
     (stroke (width 0) (type default) (color 0 0 0 0))
@@
     (pin "1")
   )
-  (symbol (lib_id "power:-BATT") (at 165.735 65.405 0) (unit 1)
-    (in_bom yes) (on_board yes)
-    (property "Reference" "#PWR0108" (id 0) (at 165.735 69.215 0)
-      (effects (font (size 1.27 1.27)) hide)
-    )
-    (property "Value" "-BATT" (id 1) (at 170.18 63.5 0))
-    (property "Footprint" "" (id 2) (at 165.735 65.405 0)
-      (effects (font (size 1.27 1.27)) hide)
-    )
-    (property "Datasheet" "" (id 3) (at 165.735 65.405 0)
-      (effects (font (size 1.27 1.27)) hide)
-    )
-    (pin "1")
-  )
   (symbol (lib_id "power:+5V") (at 183.515 102.87 90) (unit 1)
     (in_bom yes) (on_board yes) (fields_autoplaced)
@@
     )
     (property "Datasheet" "" (id 3) (at 183.515 102.87 0)
+      (effects (font (size 1.27 1.27)) hide)
+    )
+    (pin "1")
+  )
+  (symbol (lib_id "power:+BATT") (at 163.195 65.405 0) (unit 1)
+    (in_bom yes) (on_board yes)
+    (property "Reference" "#PWR0109" (id 0) (at 163.195 69.215 0)
+      (effects (font (size 1.27 1.27)) hide)
+    )
+    (property "Value" "" (id 1) (at 158.75 65.405 0))
+    (property "Footprint" "" (id 2) (at 163.195 65.405 0)
+      (effects (font (size 1.27 1.27)) hide)
+    )
+    (property "Datasheet" "" (id 3) (at 163.195 65.405 0)
+      (effects (font (size 1.27 1.27)) hide)
+    )
+    (pin "1")
+  )
+  (symbol (lib_id "power:PWR_FLAG") (at 165.735 68.58 270) (unit 1)
+    (in_bom yes) (on_board yes) (fields_autoplaced)
+    (property "Reference" "#FLG0102" (id 0) (at 167.64 68.58 0)
+      (effects (font (size 1.27 1.27)) hide)
+    )
+    (property "Value" "" (id 1) (at 168.91 68.5799 90)
+      (effects (font (size 1.27 1.27)) (justify left))
+    )
+    (property "Footprint" "" (id 2) (at 165.735 68.58 0)
+      (effects (font (size 1.27 1.27)) hide)
+    )
+    (property "Datasheet" "~" (id 3) (at 165.735 68.58 0)
       (effects (font (size 1.27 1.27)) hide)
     )
@@
     )
     (property "Datasheet" "" (id 3) (at 95.885 81.28 0)
+      (effects (font (size 1.27 1.27)) hide)
+    )
+    (pin "1")
+  )
+  (symbol (lib_id "power:PWR_FLAG") (at 163.195 68.58 90) (unit 1)
+    (in_bom yes) (on_board yes) (fields_autoplaced)
+    (property "Reference" "#FLG0101" (id 0) (at 161.29 68.58 0)
+      (effects (font (size 1.27 1.27)) hide)
+    )
+    (property "Value" "" (id 1) (at 160.02 68.5799 90)
+      (effects (font (size 1.27 1.27)) (justify left))
+    )
+    (property "Footprint" "" (id 2) (at 163.195 68.58 0)
+      (effects (font (size 1.27 1.27)) hide)
+    )
+    (property "Datasheet" "~" (id 3) (at 163.195 68.58 0)
       (effects (font (size 1.27 1.27)) hide)
     )
@@
     (pin "1")
   )
+  (symbol (lib_id "power:+9V") (at 169.545 80.01 270) (unit 1)
+    (in_bom yes) (on_board yes) (fields_autoplaced)
+    (property "Reference" "#PWR0106" (id 0) (at 165.735 80.01 0)
+      (effects (font (size 1.27 1.27)) hide)
+    )
+    (property "Value" "" (id 1) (at 172.72 80.0099 90)
+      (effects (font (size 1.27 1.27)) (justify left))
+    )
+    (property "Footprint" "" (id 2) (at 169.545 80.01 0)
+      (effects (font (size 1.27 1.27)) hide)
+    )
+    (property "Datasheet" "" (id 3) (at 169.545 80.01 0)
+      (effects (font (size 1.27 1.27)) hide)
+    )
+    (pin "1")
+  )
   (symbol (lib_id "Device:R") (at 106.045 116.205 0) (mirror y) (unit 1)
     (in_bom yes) (on_board yes)
@@
     (pin "1")
   )
+  (symbol (lib_id "power:-BATT") (at 165.735 65.405 0) (unit 1)
+    (in_bom yes) (on_board yes)
+    (property "Reference" "#PWR0108" (id 0) (at 165.735 69.215 0)
+      (effects (font (size 1.27 1.27)) hide)
+    )
+    (property "Value" "" (id 1) (at 169.545 65.405 0))
+    (property "Footprint" "" (id 2) (at 165.735 65.405 0)
+      (effects (font (size 1.27 1.27)) hide)
+    )
+    (property "Datasheet" "" (id 3) (at 165.735 65.405 0)
+      (effects (font (size 1.27 1.27)) hide)
+    )
+    (pin "1")
+  )
   (symbol (lib_id "power:GND") (at 106.045 120.015 0) (mirror y) (unit 1)
     (in_bom yes) (on_board yes) (fields_autoplaced)
@@
     (pin "1")
   )
-  (symbol (lib_id "power:+BATT") (at 163.195 65.405 0) (unit 1)
-    (in_bom yes) (on_board yes)
-    (property "Reference" "#PWR0106" (id 0) (at 163.195 69.215 0)
-      (effects (font (size 1.27 1.27)) hide)
-    )
-    (property "Value" "+BATT" (id 1) (at 158.75 63.5 0))
-    (property "Footprint" "" (id 2) (at 163.195 65.405 0)
-      (effects (font (size 1.27 1.27)) hide)
-    )
-    (property "Datasheet" "" (id 3) (at 163.195 65.405 0)
-      (effects (font (size 1.27 1.27)) hide)
-    )
-    (pin "1")
-  )
   (symbol (lib_id "SSD1306-128x64_OLED:SSD1306") (at 192.405 101.6 90) (unit 1)
     (in_bom yes) (on_board yes) (fields_autoplaced)
@@
   )
   (symbol_instances
+    (path "/663eb0c5-abd8-4c3b-aa08-c370846fcb42"
+      (reference "#FLG0101") (unit 1) (value "PWR_FLAG") (footprint "")
+    )
+    (path "/26fe87f3-24cc-438c-aab3-bf79b97685b4"
+      (reference "#FLG0102") (unit 1) (value "PWR_FLAG") (footprint "")
+    )
     (path "/d946c854-5af6-4233-8458-d4111b1cccd1"
       (reference "#PWR01") (unit 1) (value "GND") (footprint "")
@@
       (reference "#PWR0105") (unit 1) (value "+5V") (footprint "")
     )
-    (path "/d94eae12-434e-41c4-b0b1-a32ff17eff68"
-      (reference "#PWR0106") (unit 1) (value "+BATT") (footprint "")
+    (path "/8dcc068a-9d92-4e58-8a3d-ab076d07da10"
+      (reference "#PWR0106") (unit 1) (value "+9V") (footprint "")
     )
     (path "/89a2b241-50ef-4a27-b56f-53b5e6216d7d"
       (reference "#PWR0107") (unit 1) (value "+5V") (footprint "")
     )
-    (path "/10a7a83c-2348-4b22-8872-e196664357ff"
+    (path "/c00190dc-5154-4ae0-afa2-421e4cfffcf8"
       (reference "#PWR0108") (unit 1) (value "-BATT") (footprint "")
     )
+    (path "/225e71fa-e9c2-427e-9477-1db6f9201dc3"
+      (reference "#PWR0109") (unit 1) (value "+BATT") (footprint "")
+    )
     (path "/f641e724-f6c6-4cc1-9573-a10a2c206448"
-      (reference "Brd1") (unit 1) (value "SSD1306") (footprint "Display:Adafruit_SSD1306")
+      (reference "Brd1") (unit 1) (value "SSD1306") (footprint "Display:Adafruit_SSD1306_No_Mounting_Holes")
     )
     (path "/4b8b957b-aa24-41cb-8992-0733069ca247"
